Commit message: Exercise 7 done!

File: Part11/part11_description/urdf/scara.urdf (robot description, URDF)
Before this commit: robot scara, 5 links, 4 joints
Links:
- added link ee_link_visual; visual cylinder length=0.3 radius=0.2
- added link link2_visual; visual cylinder length=0.3 radius=0.2
- link ee_link: geometry visual cylinder length=0.6 radius=0.05
- link link1: geometry visual box size=2.0 0.3 0.2
- link link2: geometry visual box size=2.0 0.3 0.2
Joints:
- added joint link2_to_ee_link_visual: type fixed, parent link2, child ee_link_visual, origin xyz=2 0 0
- added joint link2_to_link2_visual: type fixed, parent link2, child link2_visual, origin xyz=0 0 -0.05
- joint base_link_to_link1: origin xyz=0 0 1 -> xyz=0 0 0.65
- joint link1_to_link1_visual: origin xyz=0 0 1 -> xyz=0 0 -0.05
- joint link1_to_link2: origin xyz=0 0 1 -> xyz=2 0 0
- joint link2_to_ee_link: limit (none) -> lower=0 upper=0.6 effort=1000.0 velocity=0.5; origin xyz=0 0 1 -> xyz=2 0 0; type continuous -> prismatic
